File: parking_counter/parking_counter.kicad_pcb (KiCad board)
At the start: 2 copper layers, 91.4 x 68.6 mm, 14 parts, among them J1 IR SENSOR 1, J2 IR SENSOR 1, J3 IR SENSOR 1, J4 IR SENSOR 1, J5 Micro_SD, J6 16x2 LCD SCREEN w/I2C, J7 Comdix, U1 HiLetgo ESP-WROOM-32S

Commit message: Add files via upload
Parts:
- added R1: R10k, Resistor_THT:R_Axial_DIN0207_L6.3mm_D2.5mm_P7.62mm_Horizontal, F.Cu at (170.2, 127.0)
- added R2: R10k, Resistor_THT:R_Axial_DIN0207_L6.3mm_D2.5mm_P7.62mm_Horizontal, F.Cu at (165.1, 113.0)
- added REF**: MountingHole_2.5mm_Pad, MountingHole:MountingHole_2.5mm_Pad, F.Cu at (170.2, 76.2)
- added REF**: MountingHole_2.5mm_Pad, MountingHole:MountingHole_2.5mm_Pad, F.Cu at (94.0, 76.2)
- added REF**: MountingHole_2.5mm_Pad, MountingHole:MountingHole_2.5mm_Pad, F.Cu at (162.6, 132.1)
- added REF**: MountingHole_2.5mm_Pad, MountingHole:MountingHole_2.5mm_Pad, F.Cu at (94.0, 134.6)
- moved J6 5.08 mm to (170.2, 114.3)
- moved TP1 5.08 mm to (129.5, 129.5)
- moved J7 2.54 mm to (109.2, 116.8)
- renumbered U2 to TP4056
Routing:
- net +5V: track 152.6 -> 169.7 mm
- net Net-(J6-SCL): track 15.2 -> 29.2 mm
- net Net-(J6-SDA): track 15.2 -> 21.2 mm
- net Net-(J1-OUT): track 43.4 -> 46.3 mm
- net Net-(J7-V_IN): track 21.8 -> 24.3 mm
Other:
- board size 91.4 x 68.6 mm -> 86.4 x 68.6 mm
